Commit message: Leonardo drone contest october 2024 adjustaments

File: src/rover_description_pkg/urdf/rover.xacro (robot description, xacro)
@@ -3,6 +3,6 @@
 <xacro:include filename="$(find rover_description_pkg)/urdf/rover_macro.xacro"/>
 <xacro:include filename="$(find rover_description_pkg)/urdf/utilities.xacro"/>
-<xacro:include filename="$(find rover_description_pkg)/urdf/rover_gazebo.xacro"/>
-<xacro:include filename="$(find rover_turret_cameras)/urdf/rover_turret_macro.xacro"/>
+<!-- <xacro:include filename="$(find rover_description_pkg)/urdf/rover_gazebo.xacro"/>
+<xacro:include filename="$(find rover_turret_cameras)/urdf/rover_turret_macro.xacro"/> -->
 <xacro:arg name="is_sim" default="false"/>
 <link name="base_footprint">
@@ -16,5 +16,5 @@
 </joint>
 <xacro:rover_base_frame parent_link="base_footprint"/>
-<xacro:rover_turret parent_link="rover_turret_plate"/>
+<!-- <xacro:rover_turret parent_link="rover_turret_plate"/> -->
 <!-- if it is in simulation -->
 <xacro:if value="$(arg is_sim)">

File: src/rover_description_pkg/urdf/rover_macro.xacro (robot description, xacro)
@@ -51,5 +51,5 @@
             <parent link="base_footprint"/>
             <child link="${laser_frame}"/>
-            <origin xyz="0.0 0.0 0.23" rpy="0.0 0.0 0 "/> <!-- rpy had a 180 deg rotation on y and 0 on z -->
+            <origin xyz="0.0 0.0 0.23" rpy="0.0 3.14 0 "/> <!-- RP_lidar has a 180 deg rotation on y and 0 on z -->
         </joint>
         <link name="${laser_frame}">
@@ -61,4 +61,5 @@
         </link>
     </xacro:macro>
+<!--
     <xacro:macro name="rover_camera_realsense_d435i" params="camera_base_frame">
         <xacro:include filename="$(find realsense2_description)/urdf/_d435i.urdf.xacro"/>
@@ -72,5 +73,5 @@
         </joint>
         <link name="${camera_base_frame}"/>
-        <!-- IMU Integration -->
     </xacro:macro>
+-->
 </robot>
