Commit message: new install added to dockerfile and rs_camera file updated

File: src/rover_description_pkg/urdf/rover_gazebo.xacro (robot description, xacro)
@@ -55,10 +55,4 @@
     </link>
     <!-- IMU Integration -->
-   <joint name="camera_imu_joint" type="fixed">
-        <origin xyz="0 0 0" rpy="0 0 0"/>
-        <parent link="${camera_base_frame}"/>
-        <child link="camera_imu_frame"/>
-    </joint>
-    <link name="camera_imu_frame"/>
     <gazebo reference="camera_depth_frame">
         <sensor name="${camera_base_frame}" type="depth">
@@ -102,35 +96,4 @@
         </sensor>
     </gazebo>
-    <gazebo reference="camera_imu_frame">
-            <sensor name="camera_imu_sensor" type="imu">
-                <always_on>true</always_on>
-                <update_rate>100.0</update_rate>
-                <imu>
-                    <angular_velocity>
-                        <noise>
-                            <type>gaussian</type>
-                            <mean>0.0</mean>
-                            <stddev>0.02</stddev>
-                        </noise>
-                    </angular_velocity>
-                    <linear_acceleration>
-                        <noise>
-                            <type>gaussian</type>
-                            <mean>0.0</mean>
-                            <stddev>0.02</stddev>
-                        </noise>
-                    </linear_acceleration>
-                </imu>
-                <plugin name="camera_imu_sensor" filename="libgazebo_ros_imu.so">
-                    <ros>
-                        <namespace>/</namespace>
-                        <remapping>imu/data_raw:=/camera/imu</remapping>
-                    </ros>
-                    <update_rate>100.0</update_rate>
-                    <topicName>imu</topicName>
-                    <frameName>camera_imu_optical_frame</frameName>
-                </plugin>
-            </sensor>
-        </gazebo>
 </xacro:macro>
 <xacro:macro name="lidar_gazebo_sensor" params="laser_frame laser_topic" >

File: src/rover_description_pkg/urdf/rover_macro.xacro (robot description, xacro)
@@ -73,10 +73,4 @@
         <link name="${camera_base_frame}"/>
         <!-- IMU Integration -->
-        <joint name="camera_imu_joint" type="fixed">
-            <origin xyz="0 0 0" rpy="0 0 0"/>
-            <parent link="${camera_base_frame}"/>
-            <child link="camera_imu_frame"/>
-        </joint>
-        <link name="camera_imu_frame"/>
     </xacro:macro>
 </robot>

Commit message: rtabmap correctly configured and working on imu

File: src/rover_description_pkg/urdf/rover_gazebo.xacro (robot description, xacro)
@@ -54,4 +54,11 @@
     <link name="${camera_base_frame}">
     </link>
+    <!-- IMU Integration -->
+   <joint name="camera_imu_joint" type="fixed">
+        <origin xyz="0 0 0" rpy="0 0 0"/>
+        <parent link="${camera_base_frame}"/>
+        <child link="camera_imu_frame"/>
+    </joint>
+    <link name="camera_imu_frame"/>
     <gazebo reference="camera_depth_frame">
         <sensor name="${camera_base_frame}" type="depth">
@@ -94,52 +101,36 @@
             </plugin>
         </sensor>
-              <!-- IMU -->
-        <sensor name="${camera_base_frame}imu" type="imu">
-          <always_on>true</always_on>
-          <update_rate>400</update_rate>
-          <topic>${camera_base_frame}/imu/sample</topic>
-          <plugin name="{camera_base_frame}imu" filename="libgazebo_ros_imu_sensor.so">
-            <topicName>${camera_base_frame}/imu/sample</topicName>
-            <bodyName>${camera_base_frame}_link</bodyName>
-            <frameName>camera_imu_optical_frame</frameName>
-            <updateRateHZ>400</updateRateHZ>
-            <gaussianNoise>0.1</gaussianNoise>
-            <xyzOffset>0 0 0</xyzOffset>
-            <rpyOffset>0 0 0</rpyOffset>
-          </plugin>
-        </sensor>
-      <!-- Accel and gyro -->
-        <sensor name="{camera_base_frame}accel" type="imu">
-          <always_on>true</always_on>
-          <update_rate>20</update_rate>
-          <topic>${camera_base_frame}/accel/sample</topic>
-          <plugin name="camera_accel_plugin" filename="librealsense_gazebo_accel_sensor.so">
-            <topicName>${camera_base_frame}/accel/sample</topicName>
-            <bodyName>${camera_base_frame}_link</bodyName>
-            <updateRateHZ>20</updateRateHZ>
-            <gaussianNoise>0.1</gaussianNoise>
-            <xyzOffset>0 0 0</xyzOffset>
-            <rpyOffset>0 0 0</rpyOffset>
-            <frameName>camera_gyro_optical_frame</frameName>
-            <initialOrientationAsReference>false</initialOrientationAsReference>
-          </plugin>
-          <pose>0 0 0 0 0 0</pose>
-        </sensor>
-        <sensor name="{camera_base_frame}gyro" type="imu">
-          <always_on>true</always_on>
-          <update_rate>400</update_rate>
-          <topic>${camera_base_frame}/gyro/sample</topic>
-          <plugin name="camera_gyro_plugin" filename="librealsense_gazebo_gyro_sensor.so">
-            <topicName>${camera_base_frame}/gyro/sample</topicName>
-            <bodyName>${camera_base_frame}_link</bodyName>
-            <updateRateHZ>400</updateRateHZ>
-            <gaussianNoise>0.1</gaussianNoise>
-            <xyzOffset>0 0 0</xyzOffset>
-            <rpyOffset>0 0 0</rpyOffset>
-            <frameName>camera_gyro_optical_frame</frameName>
-            <initialOrientationAsReference>false</initialOrientationAsReference>
-          </plugin>
-        </sensor>
-    </gazebo>
+    </gazebo>
+    <gazebo reference="camera_imu_frame">
+            <sensor name="camera_imu_sensor" type="imu">
+                <always_on>true</always_on>
+                <update_rate>100.0</update_rate>
+                <imu>
+                    <angular_velocity>
+                        <noise>
+                            <type>gaussian</type>
+                            <mean>0.0</mean>
+                            <stddev>0.02</stddev>
+                        </noise>
+                    </angular_velocity>
+                    <linear_acceleration>
+                        <noise>
+                            <type>gaussian</type>
+                            <mean>0.0</mean>
+                            <stddev>0.02</stddev>
+                        </noise>
+                    </linear_acceleration>
+                </imu>
+                <plugin name="camera_imu_sensor" filename="libgazebo_ros_imu.so">
+                    <ros>
+                        <namespace>/</namespace>
+                        <remapping>imu/data_raw:=/camera/imu</remapping>
+                    </ros>
+                    <update_rate>100.0</update_rate>
+                    <topicName>imu</topicName>
+                    <frameName>camera_imu_optical_frame</frameName>
+                </plugin>
+            </sensor>
+        </gazebo>
 </xacro:macro>
 <xacro:macro name="lidar_gazebo_sensor" params="laser_frame laser_topic" >

File: src/rover_description_pkg/urdf/rover_macro.xacro (robot description, xacro)
@@ -72,4 +72,11 @@
         </joint>
         <link name="${camera_base_frame}"/>
+        <!-- IMU Integration -->
+        <joint name="camera_imu_joint" type="fixed">
+            <origin xyz="0 0 0" rpy="0 0 0"/>
+            <parent link="${camera_base_frame}"/>
+            <child link="camera_imu_frame"/>
+        </joint>
+        <link name="camera_imu_frame"/>
     </xacro:macro>
 </robot>

Commit message: new unilidar branch

File: src/rover_description_pkg/urdf/rover_gazebo.xacro (robot description, xacro)
@@ -102,5 +102,5 @@
         <child link="${laser_frame}"/>
         <!-- the lidar has been raised by 5mm with respect to its original position because of laser rays detecting ghost shapes -->
-        <origin xyz="0.0 0.0 ${0.22+0.005}" rpy="0.0 ${PI} 0.0"/>
+        <origin xyz="0.0 0.0 ${0.22+0.005}" rpy="0.0 0.0 0 "/> <!-- rpy had a 180 deg rotation on y and 0 on z -->
     </joint>
     <link name="${laser_frame}">
@@ -113,5 +113,5 @@
     <gazebo reference="${laser_frame}">
       <sensor type="ray" name="head_hokuyo_sensor">
-        <pose>0 0 0 0 -${PI} 0</pose>
+        <pose>0 0 0 0 0 0 </pose> <!-- rpy: y was -{PI} rotation on y and 0 on z-->
         <visualize>true</visualize>
         <update_rate>40</update_rate>

File: src/rover_description_pkg/urdf/rover_macro.xacro (robot description, xacro)
@@ -51,5 +51,5 @@
             <parent link="base_footprint"/>
             <child link="${laser_frame}"/>
-            <origin xyz="0.0 0.0 0.23" rpy="0.0 ${PI} 0.0"/>
+            <origin xyz="0.0 0.0 0.23" rpy="0.0 0.0 0 "/> <!-- rpy had a 180 deg rotation on y and 0 on z -->
         </joint>
         <link name="${laser_frame}">
