Commit message: Joystick launch node for simulation added

File: src/pkg/gz_migration/urdf/leo1_rtab.urdf (robot description, URDF)
Before this commit: robot leo_sim, 22 links, 21 joints
Joints:
- joint rocker_L_joint: limit lower=-0.24 upper=0.24 effort=100.0 velocity=100.0 -> lower=-0.5 upper=0.5 effort=100.0 velocity=10.0
- joint rocker_R_joint: limit lower=-0.24 upper=0.24 effort=100.0 velocity=100.0 -> lower=-0.5 upper=0.5 effort=100.0 velocity=10.0; mimic joint=rocker_L_joint -> (none)
- joint wheel_FL_joint: limit effort=2.0 velocity=6.0 -> effort=2.0 velocity=2.0
- joint wheel_FR_joint: limit effort=2.0 velocity=6.0 -> effort=2.0 velocity=2.0
- joint wheel_RL_joint: limit effort=2.0 velocity=6.0 -> effort=2.0 velocity=2.0
- joint wheel_RR_joint: limit effort=2.0 velocity=6.0 -> effort=2.0 velocity=2.0
