Commit message: object detection part removed and namespace adjsted for multi-robot tasks

File: src/pkg/rover_description_pkg/urdf/imu.urdf (robot description, URDF)
Before this commit: robot imu, 1 links, 1 joints
Links:
- removed link imu_link
Joints:
- removed joint imu_to_payload

File: src/pkg/rover_description_pkg/urdf/old/rover_gazebo.xacro (robot description, xacro)
@@ -152,8 +152,8 @@
             <legacyMode>true</legacyMode>
             <rosDebugLevel>Debug</rosDebugLevel>
-            <publishWheelTF>false</publishWheelTF>
+            <publishWheelTF>true</publishWheelTF>
             <robotNamespace>/</robotNamespace>
             <publishTf>1</publishTf>
-            <publishWheelJointState>false</publishWheelJointState>
+            <publishWheelJointState>true</publishWheelJointState>
             <alwaysOn>true</alwaysOn>
             <updateRate>100.0</updateRate>

File: src/pkg/rover_description_pkg/urdf/rover.xacro (robot description, xacro)
@@ -5,4 +5,7 @@
 <xacro:include filename="$(find rover_description_pkg)/urdf/rover_gazebo.xacro"/>
 <xacro:arg name="is_sim" default="true"/>
+<xacro:arg name="namespace" default=""/>
+<xacro:arg name="frame_prefix" default=""/>
+<xacro:arg name="tf_prefix" default=""/>
 <link name="base_footprint">
 </link>
@@ -12,13 +15,13 @@
 <xacro:if value="$(arg is_sim)">
     <xacro:rover_wheels_sim left_joint="diff_drive_l_joint" right_joint="diff_drive_r_joint"/>
-    <xacro:gazebo_diff_drive_controller left_joint="diff_drive_l_joint" right_joint="diff_drive_r_joint"/>
+    <xacro:gazebo_diff_drive_controller left_joint="diff_drive_l_joint" right_joint="diff_drive_r_joint" namespace="$(arg namespace)"/>
     <xacro:gazebo_wheel_contact/>
-    <xacro:lidar_gazebo_sensor laser_frame="lidar_link" laser_topic="scan"/>
+    <xacro:lidar_gazebo_sensor laser_frame="lidar_link" laser_topic="scan" namespace="$(arg namespace)"/>
     <!-- <xacro:rover_payload_frame payload_frame="payload_link"/> -->
-    <xacro:camera_gazebo camera_base_frame="camera_link" camera_topic="camera" camera_info_topic="camera_info"/>
+    <xacro:camera_gazebo camera_base_frame="camera_link" camera_topic="camera" camera_info_topic="camera_info" namespace="$(arg namespace)"/>
 </xacro:if>
 <!-- if it is not in simulation -->
 <xacro:unless value="$(arg is_sim)">
-    <xacro:rover_rplidar_s1 laser_frame="laser"/>
+    <xacro:lidar_gazebo_sensor laser_frame="lidar_link" laser_topic="scan" namespace="$(arg namespace)"/>
     <!-- <xacro:rover_camera_realsense_d435i camera_base_frame="camera_frame"/> -->
 </xacro:unless>

File: src/pkg/rover_description_pkg/urdf/rover_gazebo.xacro (robot description, xacro)
@@ -111,5 +111,5 @@
 </xacro:macro>
 <!-- Camera -->
-<xacro:macro name="camera_gazebo" params="camera_base_frame camera_topic camera_info_topic">
+<xacro:macro name="camera_gazebo" params="camera_base_frame camera_topic camera_info_topic namespace">
     <xacro:include filename="$(find realsense2_description)/urdf/_d435i.urdf.xacro"/>
     <!-- <xacro:sensor_d435i parent="${camera_base_frame}" use_nominal_extrinsics="true">
@@ -164,7 +164,7 @@
     <gazebo reference="${camera_base_frame}">
         <sensor name="d435_color" type="camera">
-            <topic>color/image_raw</topic>
-            <ignition_frame_id>rover/camera_link</ignition_frame_id>
-            <gz_frame_id>rover/camera_link</gz_frame_id>
+            <topic>${namespace}/color/image_raw</topic>
+            <ignition_frame_id>${namespace}/camera_link</ignition_frame_id>
+            <gz_frame_id>${namespace}/camera_link</gz_frame_id>
             <camera name="d435">
                 <camera_info_topic>color/camera_info</camera_info_topic>
@@ -223,5 +223,5 @@
 </xacro:macro>
     <!-- Gazebo Plugins -->
-<xacro:macro name="gazebo_diff_drive_controller" params="left_joint right_joint">
+<xacro:macro name="gazebo_diff_drive_controller" params="left_joint right_joint namespace">
     <gazebo>
         <plugin name="ignition::gazebo::systems::DiffDrive" filename="ignition-gazebo-diff-drive-system">
@@ -243,7 +243,7 @@
             <child_frame_id>rover/base_link</child_frame_id>
             <!-- Topics -->
-            <topic>/cmd_vel</topic>
-            <odom_topic>/odom/wheels</odom_topic>
-            <tf_topic>/tf_gazebo</tf_topic>
+            <topic>${namespace}/cmd_vel</topic>
+            <odom_topic>${namespace}/odom/wheels</odom_topic>
+            <tf_topic>${namespace}/tf_gazebo</tf_topic>
         </plugin>
         <plugin filename="ignition-gazebo-joint-state-publisher-system" name="ignition::gazebo::systems::JointStatePublisher">

File: src/pkg/rover_description_pkg/urdf/rover_macro.xacro (robot description, xacro)
@@ -91,5 +91,5 @@
         <child link="pole_link"/>
     </joint>
-<xacro:macro name="lidar_gazebo_sensor" params="laser_frame laser_topic">
+<xacro:macro name="lidar_gazebo_sensor" params="laser_frame laser_topic namespace">
         <joint name="lidar_to_payload" type="fixed">
             <parent link="payload_link"/>
@@ -114,6 +114,6 @@
         <sensor name='gpu_lidar' type='gpu_lidar'>
             <pose>0 0 0 0 0 0</pose>
-            <topic>${laser_topic}</topic>
-            <ignition_frame_id>rover/lidar_link</ignition_frame_id>
+            <topic>${namespace}/${laser_topic}</topic>
+            <ignition_frame_id>${namespace}/lidar_link</ignition_frame_id>
             <update_rate>30</update_rate>
             <lidar>
